File: deepsea-light-pcb.kicad_sch (KiCad schematic)
At the start: 0 parts

Commit message: Add correct pico footprint
Parts:
- added U1: Pico, MCU_RaspberryPi_and_Boards:RPi_Pico_SMD_TH, symbol MCU_RaspberryPi_and_Boards:Pico
Changed lines of the file:
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@@
 	(generator_version "9.0")
 	(paper "A4")
+	(symbol
+		(lib_id "MCU_RaspberryPi_and_Boards:Pico")
+		(at 85.09 91.44 0)
+		(unit 1)
+		(exclude_from_sim no)
+		(in_bom yes)
+		(on_board yes)
+		(dnp no)
+		(fields_autoplaced yes)
+		(property "Reference" "U1"
+			(at 85.09 59.69 0)
+			(effects
+				(font
+					(size 1.27 1.27)
+				)
+			)
+		)
+		(property "Value" "Pico"
+			(at 85.09 62.23 0)
+			(effects
+				(font
+					(size 1.27 1.27)
+				)
+			)
+		)
+		(property "Footprint" "MCU_RaspberryPi_and_Boards:RPi_Pico_SMD_TH"
+			(at 85.09 91.44 90)
+			(effects
+				(font
+					(size 1.27 1.27)
+				)
+				(hide yes)
+			)
+		)
+		(property "Datasheet" ""
+			(at 85.09 91.44 0)
+			(effects
+				(font
+					(size 1.27 1.27)
+				)
+				(hide yes)
+			)
+		)
+		(property "Description" ""
+			(at 85.09 91.44 0)
+			(effects
+				(font
+					(size 1.27 1.27)
+				)
+				(hide yes)
+			)
+		)
+		(pin "38"
+		)
+		(pin "39"
+		)
+		(pin "22"
+		)
+		(pin "36"
+		)
+		(pin "21"
+		)
+		(pin "12"
+		)
+		(pin "11"
+		)
+		(pin "10"
+		)
+		(pin "9"
+		)
+		(pin "8"
+		)
+		(pin "7"
+		)
+		(pin "6"
+		)
+		(pin "5"
+		)
+		(pin "4"
+		)
+		(pin "3"
+		)
+		(pin "2"
+		)
+		(pin "1"
+		)
+		(pin "13"
+		)
+		(pin "15"
+		)
+		(pin "14"
+		)
+		(pin "17"
+		)
+		(pin "16"
+		)
+		(pin "18"
+		)
+		(pin "19"
+		)
+		(pin "20"
+		)
+		(pin "41"
+		)
+		(pin "42"
+		)
+		(pin "43"
+		)
+		(pin "40"
+		)
+		(pin "23"
+		)
+		(pin "24"
+		)
+		(pin "28"
+		)
+		(pin "29"
+		)
+		(pin "30"
+		)
+		(pin "31"
+		)
+		(pin "35"
+		)
+		(pin "34"
+		)
+		(pin "33"
+		)
+		(pin "32"
+		)
+		(pin "27"
+		)
+		(pin "26"
+		)
+		(pin "25"
+		)
+		(pin "37"
+		)
+		(instances
+			(project ""
+				(path "/99abfaa1-ae0d-4c93-9def-8bea19834d01"
+					(reference "U1")
+					(unit 1)
+				)
+			)
+		)
+	)
 	(sheet_instances
 		(path "/"

Commit message: Placement work
Parts:
- added CN1: XT60PW-M, Deepsea_light_lib:CONN-TH_XT60PW-M, symbol Deepsea_light_lib:XT60PW-M
- added U2, U3, U4, U5: 2604-1106, Deepsea_light_lib:CONN-TH_2604-1106, symbol Deepsea_light_lib:2604-1106
Connections:
- net GND: now reaches U1.41 (SWCLK)
- net GND: now also U1.42 (GND), U1.43 (SWDIO), CN1.1 (-), U2.2, U3.2, U4.2, U5.2
- new net +24V: CN1.2 (+), U2.1, U3.1, U4.1, U5.1
- new net PULSE_SYNC: U2.4, U3.4, U4.4, U5.4
- new net RxD_B+: U2.5, U3.5, U4.5, U5.5
- new net TxD_A-: U2.6, U3.6, U4.6, U5.6
- no-connect marks 0 -> 4
Other:
- note added: "24 Volt Power Input"
- note added: "LED Connectors"
- moved on the sheet: U1
