File: deepsea-light-pcb.kicad_sch (KiCad schematic)
At the start: 8 parts, among them CN1 XT60PW-M, U1 Pico, U2 2604-1106, U3 2604-1106, U4 2604-1106, U5 2604-1106, U6 2604-1103, U7 SparkFun_RS485_Breakout

Commit message: Routing progress
Parts:
- removed U2, U3, U4, U5: 2604-1106, Deepsea_light_lib:CONN-TH_2604-1106, symbol Deepsea_light_lib:2604-1106
- added U2, U3, U4, U5: 2604-1104, Deepsea_light_lib:CONN-TH_2604-1104, symbol Deepsea_light_lib:2604-1104
Connections:
- net +24V: now also U2.1, U3.1, U4.1, U5.1
- net +5V: no longer U7.1 (3-5V)
- net LIGHT_GND: now also U2.2, U3.2, U4.2, U5.2
- net RxD_B+: now also U2.3, U3.3, U4.3, U5.3
- net TxD_A-: now also U2.4, U3.4, U4.4, U5.4
- net +3V3: now reaches U1.36 (3V3)
- net +3V3: now also U7.1 (3-5V)
- no-connect marks 28 -> 20
Other:
- note removed: "Pulse Sync Pin"

Commit message: Populate headers for fab only
Parts:
- added J1, J2: PinSocket_1x20_P2.54mm, Deepsea_light_lib:Socket_1x20_P2.54mm_NoPads, symbol Deepsea_light_lib:PinSocket_1x20_P2.54mm
- added J3: PinSocket_1x05_P2.54mm, Deepsea_light_lib:Socket_1x05_P2.54mm_NoPads, symbol Deepsea_light_lib:PinSocket_1x05_P2.54mm
- added J4: PinSocket_1x03_P2.54mm, Deepsea_light_lib:Socket_1x03_P2.54mm_NoPads, symbol Deepsea_light_lib:PinSocket_1x03_P2.54mm
- U1, U7: now left out of the parts list
Other:
- note added: "Module sockets"
- note added: "Placed by JLCPCB. U1 plugs into J1+J2, U7 into J3+J4."

Commit message: Fix header rotation
Parts:
- J1, J2, J3, J4: FT Rotation Offset (none) -> 90
Changed lines of the file:
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@@
+			)
+		)
+		(property "FT Rotation Offset" "90"
+			(at 229.87 132.08 0)
+			(hide yes)
+			(show_name no)
+			(do_not_autoplace no)
+			(effects
+				(font
+					(size 1.27 1.27)
+				)
 			)
 		)
@@
 			)
 		)
+		(property "FT Rotation Offset" "90"
+			(at 229.87 123.19 0)
+			(hide yes)
+			(show_name no)
+			(do_not_autoplace no)
+			(effects
+				(font
+					(size 1.27 1.27)
+				)
+			)
+		)
 		(instances
 			(project "deepsea-light-pcb"
@@
 			)
 		)
+		(property "FT Rotation Offset" "90"
+			(at 229.87 149.86 0)
+			(hide yes)
+			(show_name no)
+			(do_not_autoplace no)
+			(effects
+				(font
+					(size 1.27 1.27)
+				)
+			)
+		)
 		(instances
 			(project "deepsea-light-pcb"
@@
 			(at 229.87 140.97 0)
 			(hide yes)
+			(show_name no)
+			(do_not_autoplace no)
+			(effects
+				(font
+					(size 1.27 1.27)
+				)
+			)
+		)
+		(property "FT Rotation Offset" "90"
+			(at 229.87 140.97 0)
+			(hide yes)

Commit message: Fix solder connections
Connections:
- net GND: no longer U1.41 (SWCLK), U1.43 (SWDIO)
- no-connect marks 20 -> 22
Changed lines of the file:
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@@
 		)
-	)
-	(junction
-		(at 76.2 166.37)
-		(diameter 0)
-		(color 0 0 0 0)
 	)
 	(no_connect
@@
 	)
 	(no_connect
+		(at 73.66 163.83)
+	)
+	(no_connect
 		(at 58.42 143.51)
 	)
@@
 	)
 	(no_connect
+		(at 78.74 163.83)
+	)
+	(no_connect
 		(at 58.42 151.13)
 	)
@@
 	(wire
 		(pts
-			(xy 76.2 166.37) (xy 78.74 166.37)
-		)
-		(stroke
-			(width 0)
-			(type default)
-		)
-	)
-	(wire
-		(pts
 			(xy 158.75 134.62) (xy 171.45 134.62)
 		)
@@
 	(wire
 		(pts
-			(xy 76.2 166.37) (xy 73.66 166.37)
-		)
-		(stroke
-			(width 0)
-			(type default)
-		)
-	)
-	(wire
-		(pts
 			(xy 93.98 120.65) (xy 99.06 120.65)
 		)
@@
 	(wire
 		(pts
-			(xy 73.66 163.83) (xy 73.66 166.37)
-		)
-		(stroke
-			(width 0)
-			(type default)
-		)
-	)
-	(wire
-		(pts
 			(xy 50.8 53.34) (xy 63.5 53.34)
 		)
@@
 	(wire
 		(pts
-			(xy 76.2 163.83) (xy 76.2 166.37)
+			(xy 76.2 163.83) (xy 76.2 168.91)
 		)
 		(stroke
@@
 	(wire
 		(pts
-			(xy 78.74 163.83) (xy 78.74 166.37)
-		)
-		(stroke
-			(width 0)
-			(type default)
-		)
-	)
-	(wire
-		(pts
 			(xy 58.42 115.57) (xy 52.07 115.57)
 		)
 		(stroke
-			(width 0)
-			(type default)
-		)
-	)
-	(wire
-		(pts
-			(xy 76.2 166.37) (xy 76.2 168.91)
-		)
-		(stroke

Commit message: Add stemma
Parts:
- added J5: 250-104, Deepsea_light_lib:CONN-TH_4P-P3.50_250-104, symbol Deepsea_light_lib:250-104
Connections:
- net +3V3: now also J5.3
- net GND: now also J5.4
- net I2C_SDA: now reaches U1.19 (GPIO14)
- net I2C_SDA: now also J5.2
- net I2C_SCL: now reaches U1.20 (GPIO15)
- net I2C_SCL: now also J5.1
Other:
- note added: "I2C screw terminal (I2C1 on GP14/GP15) for an external INA238 power monitor"

Commit message: Add callout
Parts:
- J5: Callout (none) -> I2C Stemma / QWIIC
Changed lines of the file:
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@@
+			)
+		)
+		(property "Callout" "I2C Stemma / QWIIC"
+			(at 156.21 163.83 0)
+			(hide yes)
+			(show_name no)
+			(do_not_autoplace no)
+			(effects
+				(font
+					(size 1.27 1.27)
+				)
 			)
 		)

Commit message: Fix R/ TX Swap
Connections:
- net LIGHTS_RX: now also U7.3 (TX-O); no longer U7.2 (RX-I)
- net LIGHTS_TX: now also U7.2 (RX-I); no longer U7.3 (TX-O)
Changed lines of the file:
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@@
 		)
 	)
-	(label "LIGHTS_RX"
+	(label "LIGHTS_TX"
 		(at 52.07 50.8 0)
 		(effects
@@
 		)
 	)
-	(label "LIGHTS_TX"
+	(label "LIGHTS_RX"
 		(at 52.07 53.34 0)
 		(effects

Commit message: Replace connector
Parts:
- U2, U3, U4, U5: value 2604-1104 -> HC-JXDZFH-5.0-4P; LCSC C3309598 -> C53454557
Changed lines of the file:
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@@
 			)
 		)
-		(property "Value" "2604-1104"
+		(property "Value" "HC-JXDZFH-5.0-4P"
 			(at 180.34 105.4099 0)
 			(show_name no)
@@
 			)
 		)
-		(property "Datasheet" "https://atta.szlcsc.com/upload/public/pdf/source/20240403/5F4C121C25BCB0080802869D2966FD73.pdf"
+		(property "Datasheet" "https://jlcpcb.com/partdetail/HongCheng-HC_JXDZFH_5_04P/C53454557"
 			(at 174.244 104.013 0)
 			(hide yes)
@@
 			)
 		)
-		(property "LCSC" "C3309598"
+		(property "LCSC" "C53454557"
 			(at 176.53 104.14 0)
 			(hide yes)
@@
 			)
 		)
-		(property "Value" "2604-1104"
+		(property "Value" "HC-JXDZFH-5.0-4P"
 			(at 180.34 58.4199 0)
 			(show_name no)
@@
 			)
 		)
-		(property "Datasheet" "https://atta.szlcsc.com/upload/public/pdf/source/20240403/5F4C121C25BCB0080802869D2966FD73.pdf"
+		(property "Datasheet" "https://jlcpcb.com/partdetail/HongCheng-HC_JXDZFH_5_04P/C53454557"
 			(at 174.244 57.023 0)
 			(hide yes)
@@
 			)
 		)
-		(property "LCSC" "C3309598"
+		(property "LCSC" "C53454557"
 			(at 176.53 57.15 0)
 			(hide yes)
@@
 			)
 		)
-		(property "Value" "2604-1104"
+		(property "Value" "HC-JXDZFH-5.0-4P"
 			(at 180.34 81.2799 0)
 			(show_name no)
@@
 			)
 		)
-		(property "Datasheet" "https://atta.szlcsc.com/upload/public/pdf/source/20240403/5F4C121C25BCB0080802869D2966FD73.pdf"
+		(property "Datasheet" "https://jlcpcb.com/partdetail/HongCheng-HC_JXDZFH_5_04P/C53454557"
 			(at 174.244 79.883 0)
 			(hide yes)
@@
 			)
 		)
-		(property "LCSC" "C3309598"
+		(property "LCSC" "C53454557"
 			(at 176.53 80.01 0)
 			(hide yes)
@@
 			)
 		)
-		(property "Value" "2604-1104"
+		(property "Value" "HC-JXDZFH-5.0-4P"
 			(at 180.34 132.0799 0)
 			(show_name no)
@@
 			)
 		)
-		(property "Datasheet" "https://atta.szlcsc.com/upload/public/pdf/source/20240403/5F4C121C25BCB0080802869D2966FD73.pdf"
+		(property "Datasheet" "https://jlcpcb.com/partdetail/HongCheng-HC_JXDZFH_5_04P/C53454557"
 			(at 174.244 130.683 0)
 			(hide yes)
@@
 			)
 		)
-		(property "LCSC" "C3309598"
+		(property "LCSC" "C53454557"
 			(at 176.53 130.81 0)
 			(hide yes)
