File: deepsea-light-pcb.kicad_pcb (KiCad board)
At the start: 4 copper layers, 124.5 x 56.8 mm, 12 parts, among them CN1 XT60PW-M, J1 PinSocket_1x20_P2.54mm, J2 PinSocket_1x20_P2.54mm, J3 PinSocket_1x05_P2.54mm, J4 PinSocket_1x03_P2.54mm, U1 Pico, U2 2604-1104, U3 2604-1104, U4 2604-1104, U5 2604-1104, U6 2604-1103, U7 SparkFun_RS485_Breakout

Commit message: Add stemma connector for i2c (#6)
* Add stemma

* Fix warning

* Update connector render [skip ci]

* Add callout

* Fix warning

* Update connector render [skip ci]
Parts:
- added J5: 250-104, Deepsea_light_lib:CONN-TH_4P-P3.50_250-104, F.Cu at (208.4, 92.7)
Connections:
- U1 pad 19: unconnected-(U1-GPIO14-Pad19) -> /I2C_SDA
- U1 pad 20: unconnected-(U1-GPIO15-Pad20) -> /I2C_SCL
Routing:
- net /I2C_SDA: track 0.00 -> 65.5 mm
- net /I2C_SCL: track 0.00 -> 64.6 mm
- net +3V3: track 57.0 -> 69.8 mm
Other:
- outline, holes or cut-outs redrawn
- board text added: "3V3"
- board text added: "SCL"
- board text added: "SDA"

Commit message: Fix R/ TX Swap
Connections:
- U7 pad 2: /LIGHTS_RX -> /LIGHTS_TX
- U7 pad 3: /LIGHTS_TX -> /LIGHTS_RX
Routing:
- net /LIGHTS_TX: track 78.8 -> 77.7 mm
- net /LIGHTS_RX: track 78.7 -> 79.8 mm, vias 0 -> 1
Changed lines of the file:
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@@
 			(layers "*.Cu" "*.Mask")
 			(remove_unused_layers no)
-			(net "/LIGHTS_RX")
+			(net "/LIGHTS_TX")
 			(pinfunction "RX-I_2")
 			(pintype "input")
@@
 			(layers "*.Cu" "*.Mask")
 			(remove_unused_layers no)
-			(net "/LIGHTS_TX")
+			(net "/LIGHTS_RX")
 			(pinfunction "TX-O_3")
 			(pintype "output")
@@
 	)
 	(segment
-		(start 195.44 92.3)
-		(end 191.75 92.3)
+		(start 189.21 94.84)
+		(end 195.44 94.84)
 		(width 0.2)
 		(layer "In1.Cu")
@@
 	)
 	(segment
-		(start 191.75 92.3)
-		(end 185.55 98.5)
+		(start 185.55 98.5)
+		(end 189.21 94.84)
 		(width 0.2)
 		(layer "In1.Cu")
@@
 	)
 	(segment
-		(start 162.45 73.7)
-		(end 162.45 97.5)
+		(start 186.65 100)
+		(end 194.35 92.3)
 		(width 0.2)
-		(layer "In1.Cu")
+		(layer "F.Cu")
 		(net "/LIGHTS_RX")
 	)
 	(segment
-		(start 172.35 100)
-		(end 186.65 100)
+		(start 194.35 92.3)
+		(end 195.44 92.3)
 		(width 0.2)
-		(layer "In1.Cu")
+		(layer "F.Cu")
+		(net "/LIGHTS_RX")
+	)
+	(via
+		(at 186.65 100)
+		(size 0.7)
+		(drill 0.3)
+		(layers "F.Cu" "B.Cu")
 		(net "/LIGHTS_RX")
 	)
 	(segment
-		(start 165.95 101)
-		(end 171.35 101)
+		(start 162.45 73.7)
+		(end 162.45 97.5)
 		(width 0.2)
 		(layer "In1.Cu")
@@
 	)
 	(segment
-		(start 191.81 94.84)
-		(end 195.44 94.84)
+		(start 172.35 100)
+		(end 186.65 100)
 		(width 0.2)
 		(layer "In1.Cu")
@@
 	)
 	(segment
-		(start 150.46 61.71)
-		(end 162.45 73.7)
+		(start 165.95 101)
+		(end 171.35 101)
 		(width 0.2)
 		(layer "In1.Cu")
@@
 	)
 	(segment
-		(start 186.65 100)
-		(end 191.81 94.84)
+		(start 150.46 61.71)
+		(end 162.45 73.7)
 		(width 0.2)
 		(layer "In1.Cu")

Commit message: Replace connector
Parts:
- U2, U3, U4, U5: value 2604-1104 -> HC-JXDZFH-5.0-4P
Changed lines of the file:
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@@
 			)
 		)
-		(property "Value" "2604-1104"
+		(property "Value" "HC-JXDZFH-5.0-4P"
 			(at 0.100077 -0.000051 180)
 			(layer "F.Fab")
@@
 			)
 		)
-		(property "Datasheet" "https://atta.szlcsc.com/upload/public/pdf/source/20240403/5F4C121C25BCB0080802869D2966FD73.pdf"
+		(property "Datasheet" "https://jlcpcb.com/partdetail/HongCheng-HC_JXDZFH_5_04P/C53454557"
 			(at 0 0 180)
 			(layer "F.Fab")
@@
 			)
 		)
-		(property "LCSC" "C3309598"
+		(property "LCSC" "C53454557"
 			(at 0 0 180)
 			(unlocked yes)
@@
 		)
 		(embedded_fonts no)
-		(model "Deepsea_light_dir/CONN-TH_2604-1104.step"
+		(model "${KIPRJMOD}/Deepsea_light_lib/Deepsea_light_lib/Deepsea_light_dir/HC-JXDZFH-5.0-4P.step"
 			(offset
-				(xyz 1.5 -9 -3)
+				(xyz 0 0 0)
 			)
 			(scale
@@
 			)
 			(rotate
-				(xyz -0 -0 -0)
+				(xyz 0 0 0)
 			)
 		)
@@
 			)
 		)
-		(property "Value" "2604-1104"
+		(property "Value" "HC-JXDZFH-5.0-4P"
 			(at 0 0 180)
 			(layer "F.Fab")
@@
 			)
 		)
-		(property "Datasheet" "https://atta.szlcsc.com/upload/public/pdf/source/20240403/5F4C121C25BCB0080802869D2966FD73.pdf"
+		(property "Datasheet" "https://jlcpcb.com/partdetail/HongCheng-HC_JXDZFH_5_04P/C53454557"
 			(at 0 0 180)
 			(layer "F.Fab")
@@
 			)
 		)
-		(property "LCSC" "C3309598"
+		(property "LCSC" "C53454557"
 			(at 0 0 180)
 			(unlocked yes)
@@
 		)
 		(embedded_fonts no)
-		(model "Deepsea_light_dir/CONN-TH_2604-1104.step"
+		(model "${KIPRJMOD}/Deepsea_light_lib/Deepsea_light_lib/Deepsea_light_dir/HC-JXDZFH-5.0-4P.step"
 			(offset
-				(xyz 1.5 -9 -3)
+				(xyz 0 0 0)
 			)
 			(scale
@@
 			)
 			(rotate
-				(xyz -0 -0 -0)
+				(xyz 0 0 0)
 			)
 		)
@@
 			)
 		)
-		(property "Value" "2604-1104"
+		(property "Value" "HC-JXDZFH-5.0-4P"
 			(at 0 0 180)
 			(layer "F.Fab")
@@
 			)
 		)
-		(property "Datasheet" "https://atta.szlcsc.com/upload/public/pdf/source/20240403/5F4C121C25BCB0080802869D2966FD73.pdf"
+		(property "Datasheet" "https://jlcpcb.com/partdetail/HongCheng-HC_JXDZFH_5_04P/C53454557"
 			(at 0 0 180)
 			(layer "F.Fab")
@@
 			)
 		)
-		(property "LCSC" "C3309598"
+		(property "LCSC" "C53454557"
 			(at 0 0 180)
 			(unlocked yes)
@@
 		)
 		(embedded_fonts no)
-		(model "Deepsea_light_dir/CONN-TH_2604-1104.step"
+		(model "${KIPRJMOD}/Deepsea_light_lib/Deepsea_light_lib/Deepsea_light_dir/HC-JXDZFH-5.0-4P.step"
 			(offset
-				(xyz 1.5 -9 -3)
+				(xyz 0 0 0)
 			)
 			(scale
@@
 			)
 			(rotate
-				(xyz -0 -0 -0)
+				(xyz 0 0 0)
 			)
 		)
@@
 			)
 		)
-		(property "Value" "2604-1104"
+		(property "Value" "HC-JXDZFH-5.0-4P"
 			(at -0.000013 0.099949 180)
 			(layer "F.Fab")
@@
 			)
 		)
-		(property "Datasheet" "https://atta.szlcsc.com/upload/public/pdf/source/20240403/5F4C121C25BCB0080802869D2966FD73.pdf"
+		(property "Datasheet" "https://jlcpcb.com/partdetail/HongCheng-HC_JXDZFH_5_04P/C53454557"
 			(at 0 0 180)
 			(layer "F.Fab")
@@
 			)
 		)
-		(property "LCSC" "C3309598"
+		(property "LCSC" "C53454557"
 			(at 0 0 180)
 			(unlocked yes)
@@
 		)
 		(embedded_fonts no)
-		(model "Deepsea_light_dir/CONN-TH_2604-1104.step"
+		(model "${KIPRJMOD}/Deepsea_light_lib/Deepsea_light_lib/Deepsea_light_dir/HC-JXDZFH-5.0-4P.step"
 			(offset
-				(xyz 1.9 -9 -3)
+				(xyz 0 0 0)
 			)
 			(scale
@@
 			)
 			(rotate
-				(xyz -0 -0 -0)
+				(xyz 0 0 0)
 			)
 		)
